File: KiCad/internal_clock.kicad_sch (KiCad schematic)
At the start: 8 parts, among them U1 TL074

Commit message: new logo, via correction, gerber
Other:
- company: Dirty Dream - Nathanael Noir -> © Dirty Dream - Nathanael Noir
- title: 8 Step Sequencer -> Modulo-8 Seqencer
Changed lines of the file:
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@@
 	(paper "A4")
 	(title_block
-		(title "8 Step Sequencer")
-		(date "2026-03-21")
+		(title "Modulo-8 Seqencer")
+		(date "2026-04-02")
 		(rev "v1.0")
-		(company "Dirty Dream - Nathanael Noir")
+		(company "© Dirty Dream - Nathanael Noir")
 	)
 	(rectangle
