File: KiCad/power.kicad_sch (KiCad schematic)
At the start: 13 parts, among them J6 10-pin power header, U1 TL074

Commit message: fixing some errors in schematics; first component placement
Connections:
- net +12V: now also FB1.2, J6.10 (Pin_10), J6.9 (Pin_9)
- net -12V: now also FB2.2, J6.1 (Pin_1), J6.2 (Pin_2)
Changed lines of the file:
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@@
+		)
+	)
+	(label "+12V"
+		(at 58.42 39.37 0)
+		(effects
+			(font
+				(size 1.27 1.27)
+			)
+			(justify left bottom)
+		)
+	)
+	(label "-12V"
+		(at 59.69 57.15 0)
+		(effects
+			(font
+				(size 1.27 1.27)
+			)
+			(justify left bottom)
 		)
 	)

Commit message: new logo, via correction, gerber
Other:
- company: Dirty Dream - Nathanael Noir -> © Dirty Dream - Nathanael Noir
- title: 8 Step Sequencer -> Modulo-8 Seqencer
Changed lines of the file:
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@@
 	(paper "A4")
 	(title_block
-		(title "8 Step Sequencer")
-		(date "2026-03-21")
+		(title "Modulo-8 Seqencer")
+		(date "2026-04-02")
 		(rev "v1.0")
-		(company "Dirty Dream - Nathanael Noir")
+		(company "© Dirty Dream - Nathanael Noir")
 	)
 	(rectangle
