File: KiCad/switches_led.kicad_sch (KiCad schematic)
At the start: 70 parts, among them Q2 MMBT3904, Q3 MMBT3904, Q4 MMBT3904, Q5 MMBT3904, Q6 MMBT3904, Q7 MMBT3904, Q8 MMBT3904, Q9 MMBT3904, U3 CD4017BE

Commit message: new logo, via correction, gerber
Other:
- company: Dirty Dream - Nathanael Noir -> © Dirty Dream - Nathanael Noir
- title: 8 Step Sequencer -> Modulo-8 Seqencer
Changed lines of the file:
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@@
 	(paper "A4")
 	(title_block
-		(title "8 Step Sequencer")
-		(date "2026-03-21")
+		(title "Modulo-8 Seqencer")
+		(date "2026-04-02")
 		(rev "v1.0")
-		(company "Dirty Dream - Nathanael Noir")
+		(company "© Dirty Dream - Nathanael Noir")
 	)
 	(junction
